File: hx8kevb-sdram.kicad_pcb (KiCad board)
At the start: 2 copper layers, 56 x 74.1 mm, 17 parts, among them P1 CONN_02X20, P2 CONN_02X20, P3 CONN_01X03, P4 CONN_01X12, P5 CONN_01X09, U1 AS4C16M16

Commit message: rev b
Connections:
- P1 pad 2: Net-(P1-Pad2) -> (no net)
- P1 pad 26: Net-(P1-Pad26) -> (no net)
- P2 pad 10: /GPIO6 -> /DQ0
- P2 pad 11: /GPIO7 -> (no net)
- P2 pad 12: /DQ0 -> (no net)
- P5 pad 3: /GPIO7 -> (no net)
- P5 pad 4: /GPIO6 -> (no net)
- U1 pad 40: Net-(U1-Pad40) -> (no net)
Routing:
- net /GPIO7: track 41.9 -> 0.00 mm
- net /GPIO6: track 35.8 -> 0.00 mm
- net /DQ0: track 21.1 -> 20.1 mm
Other:
- board text added: "hx8k sdram rev b nn 2016"
- board text removed: "hx8k sdram rev a nn 2016"
