File: hx8kevb-sdram.sch (KiCad schematic (older format))
At the start: 17 parts, among them P1 CONN_02X20, P2 CONN_02X20, P3 CONN_01X03, P4 CONN_01X12, P5 CONN_01X09, U1 AS4C16M16

Commit message: rev b
Connections:
- net DQ0: now also P2.10 (P10); no longer P2.12 (P12)
- net GPIO6: no longer P2.10 (P10)
- net GPIO7: no longer P2.11 (P11)
- no-connect marks 3 -> 5
Changed lines of the file:
@@
 Text Label 3500 2600 0    60   ~ 0
 DQ2
-Text Label 3500 2500 0    60   ~ 0
+Text Label 3450 2400 0    60   ~ 0
 DQ0
 Text Label 4900 2600 2    60   ~ 0
@@
 Text Label 4950 2200 2    60   ~ 0
 GPIO3
-Text Label 3450 2400 0    60   ~ 0
-GPIO6
 Text Label 4950 2400 2    60   ~ 0
 GPIO5
-Text Label 4950 2500 2    60   ~ 0
-GPIO7
 Text Label 7200 5650 2    60   ~ 0
 GPIO6
@@
 	6700 5650 7200 5650
 Wire Wire Line
-	4450 2500 4950 2500
-Wire Wire Line
 	4450 2400 4950 2400
 Wire Wire Line
@@
 Wire Wire Line
 	4450 2600 4900 2600
-Wire Wire Line
-	3950 2500 3500 2500
 Wire Wire Line
 	3950 2600 3500 2600
@@
 Connection ~ 3800 1650
 NoConn ~ 2150 2000
+NoConn ~ 3950 2500
+NoConn ~ 4450 2500
 $EndSCHEMATC
